File: KiCAD/Greaseweazle.sch (KiCad schematic (older format))
At the start: 38 parts, among them J1 USB_B_Micro, J2 PROG, J3 POWER, J4 Conn_02x17_Odd_Even, U1 SPX3819M5-L-3-3, U2 STM32F103C8Tx, Y1 8M

Commit message: Kicad : 0.2 with additional regulator footprint, DISKCHANGE signal and ID jumpers
Parts:
- added JP1: ID0, Jumper:SolderJumper-3_P1.3mm_Open_RoundedPad1.0x1.5mm, symbol Jumper:SolderJumper_3_Open
- added JP2: ID1, Jumper:SolderJumper-3_P1.3mm_Open_RoundedPad1.0x1.5mm, symbol Jumper:SolderJumper_3_Open
- added R4: 1k, Resistor_SMD:R_0805_2012Metric, symbol Device:R_Small
- added U3: XC6206PxxxMR, Package_TO_SOT_SMD:SOT-23, symbol Regulator_Linear:XC6206PxxxMR
- J1: footprint Sassa:USB-MICRO-B -> Connector_USB:USB_Micro-B_Molex-105017-0001
Connections:
- net +3V3: now also J2.5 (Pin_5), JP1.3 (B), JP2.3 (B), U3.2 (VO); no longer J2.2 (Pin_2)
- net +5V: now also R4.1, U3.3 (VI)
- net BOOT0: now also J2.4 (Pin_4); no longer J2.3 (Pin_3)
- net GND: now also JP1.1 (A), JP2.1 (A), U3.1 (GND)
- net SWCLK: now also J2.2 (Pin_2); no longer J2.4 (Pin_4)
- net SWDIO: now also J2.3 (Pin_3); no longer J2.5 (Pin_5)
- net _DSKCHG: now reaches U2.29 (PA8)
- net _DSKCHG: now also J4.34 (Pin_34), R4.2
- net ID0: now reaches U2.3 (PC14)
- net ID0: now also JP1.2 (C)
- net ID1: now reaches U2.4 (PC15)
- net ID1: now also JP2.2 (C)
- no-connect marks 12 -> 9
Other:
- note added: "Board ID"
- note added: "Floppy power"
- note added: "alternative footprint"
- moved on the sheet: C6, C7, C8, C9, D1, J2, J3, J4, R2, RN1
